File: usbc pd airsoft module.kicad_pcb (KiCad board)
At the start: 2 copper layers, 135 x 21 mm, 98 parts, among them J1 USB_C_Receptacle_USB2.0_16P, J2 BALANCE 3S (JST-XH 4P), Q1 2N7002, Q2 DMP3099L, Q3 2N7002, U1 CH224K, U2 TPD2E2U06DCK, U3 BQ25798RQMR, U4 BQ7692003PWR, U5 AP7381-33SA-7, U6 STM32F042F6P6

Commit message: Rev B: charge through the balance plug, J2 pinout fix, cell LEDs + LED board
Main board (Rev B):
- Pack connects only through the JST-XH balance plug J2; Deans pads TP1-TP4 and the MAIN_P copper removed
- F1 is now a 2.5 A fast 1206 fuse (AEM F1206SB2500V032TM, LCSC C310999) between J2 pack+ and the charger
- J2 pin order matches the real pack plug: pin 1 = pack+ (red), pin 4 = pack- (black); 3D model added
- Three cell-LED wire pads A/B/C (TP13-TP15, 100R each) on PA1/PA3/PA0, freed from unused /INT, PG, ALERT
- JP2, logos and back text carried into the layout scripts; LAVADY logo reference hidden (was G***)
- ERC 0, verify.py 208/208, DRC 0 errors / 0 unconnected / 0 parity

Firmware: pauses the charger ~0.75 s every 10 s (4 s near full) for clean cell readings through the
balance wires; charlieplexed red/green cell LEDs (red = charging, green = full, red blink = fault).

LED board (new, led_board/): 20 x 10 mm, three Kingbright KPHBM-2012SURKCGKC red/green LEDs (S1-S3),
wire pads A/B/C, M2 holes; schematic checked pin by pin (verify_led.py 18/18), routed, DRC 0.

App: hints say balance plug instead of Deans. Production files for both boards via
layout_work/make_production.py. Docs updated.

Co-Authored-By: Claude Opus 5.5 <noreply@anthropic.com>
Parts:
- removed TP1: BATT IN +, Connector_Wire:SolderWirePad_1x01_SMD_3x6mm
- removed TP2: GUN OUT +, Connector_Wire:SolderWirePad_1x01_SMD_3x6mm
- removed TP3: BATT IN -, Connector_Wire:SolderWirePad_1x01_SMD_3x6mm
- removed TP4: GUN OUT -, Connector_Wire:SolderWirePad_1x01_SMD_3x6mm
- added LOGO*: LOGO, LAVADY:LAVADY logo 15x5.7mm, F.Cu at (207.1, 111.5)
- added LOGO*: LOGO, LAVADY:LAVADY logo 20x7.7mm, B.Cu at (196.2, 111.2)
- added R27: 100R, Resistor_SMD:R_0402_1005Metric, F.Cu at (113.0, 116.4)
- added R28: 100R, Resistor_SMD:R_0402_1005Metric, F.Cu at (115.5, 116.4)
- added R29: 100R, Resistor_SMD:R_0402_1005Metric, F.Cu at (118.0, 116.4)
- added TP13: LED_A, TestPoint:TestPoint_Pad_D1.5mm, F.Cu at (113.0, 114.0)
- added TP14: LED_B, TestPoint:TestPoint_Pad_D1.5mm, F.Cu at (115.5, 114.0)
- added TP15: LED_C, TestPoint:TestPoint_Pad_D1.5mm, F.Cu at (118.0, 114.0)
- F1: value 3A 32V fast -> 2.5A 32V fast
Connections:
- F1 pad 1: /MAIN_P -> /PACK_P
- J2 pad 1: /GND -> /PACK_P
- J2 pad 2: /CELL1_P -> /CELL2_P
- J2 pad 3: /CELL2_P -> /CELL1_P
- J2 pad 4: /PACK_P -> /GND
- U6 pad 6: /CHG_INT_N -> /CLED_C
- U6 pad 7: /PD_PG -> /CLED_A
- U6 pad 9: /BMS_ALERT -> /CLED_B
Routing:
- net /BMS_ALERT: track 87.7 -> 4.01 mm, vias 2 -> 0
- net /CHG_INT_N: track 65.1 -> 9.03 mm, vias 2 -> 0
- net /CLED_A: track 0.00 -> 30.2 mm, vias 0 -> 2
- net /CLED_B: track 0.00 -> 22.5 mm
- net /PACK_P: track 29.1 -> 47.3 mm, vias 2 -> 4
- net /CLED_C: track 0.00 -> 16.8 mm
- net /MAIN_P: track 11.0 -> 0.00 mm, vias 4 -> 0
- net /PD_PG: track 13.5 -> 4.06 mm
- net /LED_C: track 0.00 -> 1.89 mm
- net /LED_B: track 0.00 -> 1.89 mm
- net /LED_A: track 0.00 -> 1.89 mm
- net /CELL1_P: track 12.9 -> 11.2 mm, vias 2 -> 0
- net /GND: track 54.8 -> 55.5 mm, vias 104 -> 111
- net /CELL2_P: track 11.9 -> 11.3 mm
- net /FAST_CHG_N: track 3.44 -> 2.84 mm
- removed copper zone on B.Cu, net /MAIN_P
Other:
- board text added: "<desighned by Fluff>"
- board text added: "A"
- board text added: "B"
- board text added: "C"
