File: usbc pd airsoft module.kicad_sch (KiCad schematic)
At the start: 98 parts, among them J1 USB_C_Receptacle_USB2.0_16P, J2 BALANCE 3S (JST-XH 4P), Q1 2N7002, Q2 DMP3099L, Q3 2N7002, U1 CH224K, U2 TPD2E2U06DCK, U3 BQ25798RQMR, U4 BQ7692003PWR, U5 AP7381-33SA-7, U6 STM32F042F6P6

Commit message: Rev B: charge through the balance plug, J2 pinout fix, cell LEDs + LED board
Main board (Rev B):
- Pack connects only through the JST-XH balance plug J2; Deans pads TP1-TP4 and the MAIN_P copper removed
- F1 is now a 2.5 A fast 1206 fuse (AEM F1206SB2500V032TM, LCSC C310999) between J2 pack+ and the charger
- J2 pin order matches the real pack plug: pin 1 = pack+ (red), pin 4 = pack- (black); 3D model added
- Three cell-LED wire pads A/B/C (TP13-TP15, 100R each) on PA1/PA3/PA0, freed from unused /INT, PG, ALERT
- JP2, logos and back text carried into the layout scripts; LAVADY logo reference hidden (was G***)
- ERC 0, verify.py 208/208, DRC 0 errors / 0 unconnected / 0 parity

Firmware: pauses the charger ~0.75 s every 10 s (4 s near full) for clean cell readings through the
balance wires; charlieplexed red/green cell LEDs (red = charging, green = full, red blink = fault).

LED board (new, led_board/): 20 x 10 mm, three Kingbright KPHBM-2012SURKCGKC red/green LEDs (S1-S3),
wire pads A/B/C, M2 holes; schematic checked pin by pin (verify_led.py 18/18), routed, DRC 0.

App: hints say balance plug instead of Deans. Production files for both boards via
layout_work/make_production.py. Docs updated.

Co-Authored-By: Claude Opus 5.5 <noreply@anthropic.com>
Parts:
- removed TP1: BATT IN +, Connector_Wire:SolderWirePad_1x01_SMD_3x6mm, symbol Connector:TestPoint
- removed TP2: GUN OUT +, Connector_Wire:SolderWirePad_1x01_SMD_3x6mm, symbol Connector:TestPoint
- removed TP3: BATT IN -, Connector_Wire:SolderWirePad_1x01_SMD_3x6mm, symbol Connector:TestPoint
- removed TP4: GUN OUT -, Connector_Wire:SolderWirePad_1x01_SMD_3x6mm, symbol Connector:TestPoint
- added R27, R28, R29: 100R, Resistor_SMD:R_0402_1005Metric, symbol Device:R_Small
- added TP13: LED_A, TestPoint:TestPoint_Pad_D1.5mm, symbol Connector:TestPoint
- added TP14: LED_B, TestPoint:TestPoint_Pad_D1.5mm, symbol Connector:TestPoint
- added TP15: LED_C, TestPoint:TestPoint_Pad_D1.5mm, symbol Connector:TestPoint
- F1: value 3A 32V fast -> 2.5A 32V fast; MPN Littelfuse 1206SFF300F/32 (any 3A >=32V 1206 fast fuse) -> AEM F1206SB2500V032TM (LCSC C310999), 2.5A fast, 50A breaki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
- J2: Note Pin1 = pack NEGATIVE (black). CHECK your pack! -> Pin4 = pack NEGATIVE (black), pin1 = pack + (red): set by t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
Connections:
- net MAIN_P is gone; now on net PACK_P: F1.1
- net BMS_ALERT: no longer U6.9 (PA3)
- net CELL1_P: now also J2.3 (Pin_3); no longer J2.2 (Pin_2)
- net CELL2_P: now also J2.2 (Pin_2); no longer J2.3 (Pin_3)
- net CHG_INT_N: no longer U6.6 (PA0)
- net GND: now also J2.4 (Pin_4); no longer J2.1 (Pin_1)
- net PACK_P: now also J2.1 (Pin_1); no longer J2.4 (Pin_4)
- net PD_PG: no longer U6.7 (PA1)
- new net CLED_A: R27.1, U6.7 (PA1)
- new net CLED_B: R28.1, U6.9 (PA3)
- new net CLED_C: R29.1, U6.6 (PA0)
- new net LED_A: R27.2, TP13.1
- new net LED_B: R28.2, TP14.1
- new net LED_C: R29.2, TP15.1
Other:
- note added: "3S per datasheet Table 9-2: VC5-VC4 = cell3, VC4=VC3=VC2 shorted, VC2-VC1 = cell2, VC1-VC0 = cell1. Rc=56R / Cc=1uF cell filters -> ~37mA internal balancing (datasheet min Rc 40R, max 50mA) (never balance adjacent cells together). SRP/SRN to VSS (no coulomb counter), CHG/DSG unused. Sits in SHIP mode (~0.6uA) when idle. Balance lead also carries the charge current (pins 1 and 4): firmware pauses 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"
- note added: "6. CHARGE PATH (through the balance plug J2)"
- note added: "7. CELL LEDs (3 wire pads near the USB-C, charlieplexed)"
- note added: "PF0/PF1 = I2C1 SDA/SCL (AF1). PA11/PA12 remapped onto pins 17/18 for USB (SYSCFG PA11_PA12_RMP). PA1/PA3/PA0 = charlieplexed cell LEDs A/B/C (pads TP13-15). Charger /INT, CH224K PG and BMS ALERT are not wired to the MCU (firmware polls I2C). PA2 CHG_EN, PA4 BMS boot, PA5 VBUS/11 ADC, PA6 LED, PA7 PWR_HOLD. PB1 = FAST_CHG_N (JP2 to GND, internal pull-up): open = slow charge (default), bridged = fa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"
- note added: "Remote LED board: three 2-pin red/green bi-colour LEDs (one per cell), wired in a triangle: cell 1 between LED_A-LED_B, cell 2 between LED_B-LED_C, cell 3 between LED_C-LED_A. Red LED anode on the first pad of the pair, green anode on the second. 3 wires, no GND wire. Red = cell charging, green = cell full; lit only while charging. ~6 mA peak, 1/3 duty."
- note added: "The pack connects ONLY through the JST-XH balance plug J2 (no Deans / main-lead pads). Charge current: J2 pin 1 (pack +) -> F1 2.5A fast -> BAT_P (charger), return via J2 pin 4 (GND). J2 pin order follows the pack's plug: its black wire lands on header pin 4 (checked on the real pack). F1 protects the thin balance wires: a board short would otherwise burn them inside the stock. Max charge 1.4 A (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"
- note removed: "3S per datasheet Table 9-2: VC5-VC4 = cell3, VC4=VC3=VC2 shorted, VC2-VC1 = cell2, VC1-VC0 = cell1. Rc=56R / Cc=1uF cell filters -> ~37mA internal balancing (datasheet min Rc 40R, max 50mA) (never balance adjacent cells together). SRP/SRN to VSS (no coulomb counter), CHG/DSG unused. Sits in SHIP mode (~0.6uA) when idle. Balance lead = SENSE ONLY (charging goes through the Deans main lead), so rea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"
- note removed: "6. BATTERY + GUN (Deans T-plug pass-through)"
- note removed: "Deans pigtail from the battery -> BATT IN pads, Deans pigtail to the gun -> GUN OUT pads. Place each IN/OUT pair side by side and join them with a short, solid copper pour on BOTH layers + stitching vias (or solder both wires to one pad): gun current never crosses the board. Charger taps MAIN_P through F1 (3A). Balance plug J2 is sense-only. Field check: unplug from the gun, plug a phone (USB-C O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"
- note removed: "PF0/PF1 = I2C1 SDA/SCL (AF1). PA11/PA12 remapped onto pins 17/18 for USB (SYSCFG PA11_PA12_RMP). PA0 /INT charger, PA1 PD_PG, PA2 CHG_EN, PA3 ALERT, PA4 BMS boot, PA5 VBUS/11 ADC, PA6 LED, PA7 PWR_HOLD. PB1 = FAST_CHG_N (JP2 to GND, internal pull-up): open = slow charge (default), bridged = fast charge. Bridge JP1 + plug USB = ST ROM DFU bootloader. Backup: ST-Link on test pads TP5 SWDIO, TP6 SWC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"
- moved on the sheet: F1
